File: Themistor_Breakout.sch (EAGLE design)
At the start: 8 parts

Commit message: Added mounting holes to thermistor breakout
Parts:
- added H1, H2: MOUNT-PAD-ROUND3.6, holes:MOUNT-PAD-ROUND3.6
Connections:
- net GND: now also H1.MOUNT, H2.MOUNT
Changed lines of the file:
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@@
 <part name="J6" library="SparkFun-Connectors" library_urn="urn:adsk.eagle:library:513" deviceset="CONN_02" device="3.5MM" package3d_urn="urn:adsk.eagle:package:38050/1"/>
 <part name="J7" library="SparkFun-Connectors" library_urn="urn:adsk.eagle:library:513" deviceset="CONN_02" device="3.5MM" package3d_urn="urn:adsk.eagle:package:38050/1"/>
+<part name="H1" library="holes" library_urn="urn:adsk.eagle:library:237" deviceset="MOUNT-PAD-ROUND" device="3.6" package3d_urn="urn:adsk.eagle:package:14284/1"/>
+<part name="H2" library="holes" library_urn="urn:adsk.eagle:library:237" deviceset="MOUNT-PAD-ROUND" device="3.6" package3d_urn="urn:adsk.eagle:package:14284/1"/>
 </parts>
 <sheets>
@@
 <instance part="J6" gate="G$1" x="78.74" y="63.5"/>
 <instance part="J7" gate="G$1" x="78.74" y="53.34"/>
+<instance part="H1" gate="G$1" x="83.82" y="25.4"/>
+<instance part="H2" gate="G$1" x="83.82" y="17.78"/>
 </instances>
 <busses>
@@
 <pinref part="J7" gate="G$1" pin="1"/>
 </segment>
+<segment>
+<wire x1="81.28" y1="17.78" x2="73.66" y2="17.78" width="0.1524" layer="91"/>
+<wire x1="73.66" y1="17.78" x2="73.66" y2="15.24" width="0.1524" layer="91"/>
+<wire x1="73.66" y1="15.24" x2="73.66" y2="5.08" width="0.1524" layer="91"/>
+<wire x1="81.28" y1="25.4" x2="73.66" y2="25.4" width="0.1524" layer="91"/>
+<wire x1="73.66" y1="25.4" x2="73.66" y2="17.78" width="0.1524" layer="91"/>
+<pinref part="H2" gate="G$1" pin="MOUNT"/>
+<pinref part="H1" gate="G$1" pin="MOUNT"/>
+<label x="73.66" y="5.08" size="1.778" layer="95"/>
+</segment>
 </net>
