File: Fuel_Cell_Controller.sch (EAGLE design)
At the start: 30 parts, among them U1 MAX232PTH

Commit message: Didn't really do anything
Parts:
- added R1: 1kΩ, SparkFun-Resistors:RESISTOR0603
Connections:
- new net N$10: U$3.DIR
- new net N$11: R1.2, U$5.DIR
- net +5V: now also R1.1, U$3.VCC; no longer U$5.DIR
- net GND: now also U$3.GND
Other:
- moved on the sheet: JP1, U$3
Changed lines of the file:
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@@
 <part name="SHTSENSOR" library="FCC_parts" deviceset="SHT31-DIS" device=""/>
 <part name="JP1" library="jumper" library_urn="urn:adsk.eagle:library:252" deviceset="JP2E" device="" package3d_urn="urn:adsk.eagle:package:15452/1"/>
+<part name="R1" library="SparkFun-Resistors" deviceset="RESISTOR" device="0603" value="1kΩ"/>
 </parts>
 <sheets>
@@
 <wire x1="281.94" y1="33.02" x2="281.94" y2="-15.24" width="0.1524" layer="94"/>
 <wire x1="281.94" y1="-15.24" x2="210.82" y2="-15.24" width="0.1524" layer="94"/>
-<text x="228.6" y="-25.4" size="3.81" layer="94">TEMP/HUMID SENSOR</text>
-<wire x1="210.82" y1="-96.52" x2="304.8" y2="-96.52" width="0.1524" layer="94"/>
-<wire x1="304.8" y1="-96.52" x2="304.8" y2="-15.24" width="0.1524" layer="94"/>
-<wire x1="304.8" y1="-15.24" x2="281.94" y2="-15.24" width="0.1524" layer="94"/>
+<text x="215.9" y="-25.4" size="3.81" layer="94">TEMP/HUMID SENSOR</text>
+<wire x1="210.82" y1="-96.52" x2="281.94" y2="-96.52" width="0.1524" layer="94"/>
+<wire x1="281.94" y1="-96.52" x2="281.94" y2="-15.24" width="0.1524" layer="94"/>
 </plain>
 <instances>
@@
 <instance part="U$10" gate="G$1" x="220.98" y="53.34"/>
 <instance part="U$5" gate="G$1" x="-48.26" y="-106.68"/>
-<instance part="SHTSENSOR" gate="G$1" x="266.7" y="-58.42"/>
-<instance part="JP1" gate="1" x="248.92" y="-86.36" rot="R90"/>
+<instance part="SHTSENSOR" gate="G$1" x="254" y="-58.42"/>
+<instance part="JP1" gate="1" x="236.22" y="-86.36" rot="R90"/>
+<instance part="R1" gate="G$1" x="-78.74" y="-81.28"/>
 </instances>
 <busses>
@@
 <segment>
 <pinref part="SHTSENSOR" gate="G$1" pin="GND"/>
-<wire x1="254" y1="-48.26" x2="236.22" y2="-48.26" width="0.1524" layer="91"/>
-<label x="236.22" y="-48.26" size="1.778" layer="95"/>
+<wire x1="241.3" y1="-48.26" x2="223.52" y2="-48.26" width="0.1524" layer="91"/>
+<label x="223.52" y="-48.26" size="1.778" layer="95"/>
 </segment>
 <segment>
 <pinref part="JP1" gate="1" pin="1"/>
-<wire x1="251.46" y1="-88.9" x2="254" y2="-88.9" width="0.1524" layer="91"/>
-<wire x1="254" y1="-88.9" x2="254" y2="-91.44" width="0.1524" layer="91"/>
-<label x="254" y="-88.9" size="1.778" layer="95" rot="R270"/>
+<wire x1="238.76" y1="-88.9" x2="241.3" y2="-88.9" width="0.1524" layer="91"/>
+<wire x1="241.3" y1="-88.9" x2="241.3" y2="-91.44" width="0.1524" layer="91"/>
+<label x="241.3" y="-88.9" size="1.778" layer="95" rot="R270"/>
 </segment>
 </net>
@@
 </segment>
 <segment>
-<pinref part="U$5" gate="G$1" pin="DIR"/>
-<wire x1="-60.96" y1="-83.82" x2="-83.82" y2="-83.82" width="0.1524" layer="91"/>
-<label x="-83.82" y="-83.82" size="1.778" layer="95"/>
-</segment>
-<segment>
 <pinref part="U$5" gate="G$1" pin="VCC"/>
 <wire x1="-35.56" y1="-83.82" x2="-20.32" y2="-83.82" width="0.1524" layer="91"/>
@@
 <segment>
 <pinref part="SHTSENSOR" gate="G$1" pin="VIN"/>
-<wire x1="254" y1="-43.18" x2="236.22" y2="-43.18" width="0.1524" layer="91"/>
-<label x="236.22" y="-43.18" size="1.778" layer="95"/>
+<wire x1="241.3" y1="-43.18" x2="223.52" y2="-43.18" width="0.1524" layer="91"/>
+<label x="223.52" y="-43.18" size="1.778" layer="95"/>
 </segment>
 <segment>
 <pinref part="JP1" gate="1" pin="3"/>
-<wire x1="251.46" y1="-83.82" x2="254" y2="-83.82" width="0.1524" layer="91"/>
-<wire x1="254" y1="-83.82" x2="254" y2="-81.28" width="0.1524" layer="91"/>
-<label x="254" y="-78.74" size="1.778" layer="95" rot="R270"/>
+<wire x1="238.76" y1="-83.82" x2="241.3" y2="-83.82" width="0.1524" layer="91"/>
+<wire x1="241.3" y1="-83.82" x2="241.3" y2="-81.28" width="0.1524" layer="91"/>
+<label x="241.3" y="-78.74" size="1.778" layer="95" rot="R270"/>
+</segment>
+<segment>
+<pinref part="R1" gate="G$1" pin="1"/>
+<wire x1="-96.52" y1="-81.28" x2="-83.82" y2="-81.28" width="0.1524" layer="91"/>
+<label x="-96.52" y="-81.28" size="1.778" layer="95"/>
 </segment>
 </net>
@@
 <segment>
 <pinref part="SHTSENSOR" gate="G$1" pin="SCL"/>
-<wire x1="254" y1="-53.34" x2="236.22" y2="-53.34" width="0.1524" layer="91"/>
-<label x="236.22" y="-53.34" size="1.778" layer="95"/>
+<wire x1="241.3" y1="-53.34" x2="223.52" y2="-53.34" width="0.1524" layer="91"/>
+<label x="223.52" y="-53.34" size="1.778" layer="95"/>
 </segment>
 </net>
@@
 <segment>
 <pinref part="SHTSENSOR" gate="G$1" pin="ADR"/>
-<wire x1="254" y1="-63.5" x2="236.22" y2="-63.5" width="0.1524" layer="91"/>
-<label x="236.22" y="-63.5" size="1.778" layer="95"/>
+<wire x1="241.3" y1="-63.5" x2="223.52" y2="-63.5" width="0.1524" layer="91"/>
+<label x="223.52" y="-63.5" size="1.778" layer="95"/>
 </segment>
 <segment>
 <pinref part="JP1" gate="1" pin="2"/>
-<wire x1="251.46" y1="-86.36" x2="274.32" y2="-86.36" width="0.1524" layer="91"/>
-<label x="264.16" y="-86.36" size="1.778" layer="95"/>
+<wire x1="238.76" y1="-86.36" x2="261.62" y2="-86.36" width="0.1524" layer="91"/>
+<label x="251.46" y="-86.36" size="1.778" layer="95"/>
 </segment>
 </net>
@@
 <segment>
 <pinref part="SHTSENSOR" gate="G$1" pin="RST"/>
-<wire x1="254" y1="-68.58" x2="236.22" y2="-68.58" width="0.1524" layer="91"/>
-<label x="236.22" y="-68.58" size="1.778" layer="95"/>
+<wire x1="241.3" y1="-68.58" x2="223.52" y2="-68.58" width="0.1524" layer="91"/>
+<label x="223.52" y="-68.58" size="1.778" layer="95"/>
 </segment>
 </net>
@@
 <segment>
 <pinref part="SHTSENSOR" gate="G$1" pin="SDA"/>
-<wire x1="254" y1="-58.42" x2="236.22" y2="-58.42" width="0.1524" layer="91"/>
-<label x="236.22" y="-58.42" size="1.778" layer="95"/>
+<wire x1="241.3" y1="-58.42" x2="223.52" y2="-58.42" width="0.1524" layer="91"/>
+<label x="223.52" y="-58.42" size="1.778" layer="95"/>
 </segment>
 </net>
@@
 <wire x1="-71.12" y1="-38.1" x2="-99.06" y2="-38.1" width="0.1524" layer="91"/>
 <label x="-99.06" y="-38.1" size="1.778" layer="95"/>
+</segment>
+</net>
+<net name="N$11" class="0">
+<segment>
+<pinref part="R1" gate="G$1" pin="2"/>
+<wire x1="-73.66" y1="-81.28" x2="-66.04" y2="-81.28" width="0.1524" layer="91"/>
+<wire x1="-66.04" y1="-81.28" x2="-66.04" y2="-83.82" width="0.1524" layer="91"/>
+<pinref part="U$5" gate="G$1" pin="DIR"/>
+<wire x1="-66.04" y1="-83.82" x2="-60.96" y2="-83.82" width="0.1524" layer="91"/>
 </segment>
 </net>
@@
 </plain>
 <instances>
-<instance part="U$3" gate="G$1" x="10.16" y="48.26"/>
+<instance part="U$3" gate="G$1" x="-5.08" y="48.26"/>
 <instance part="U$4" gate="G$1" x="81.28" y="66.04"/>
 <instance part="U$7" gate="G$1" x="134.62" y="58.42"/>
@@
 <segment>
 <pinref part="U$4" gate="G$1" pin="ANODE"/>
-<wire x1="66.04" y1="71.12" x2="35.56" y2="71.12" width="0.1524" layer="91"/>
-<label x="35.56" y="71.12" size="1.778" layer="95"/>
+<wire x1="66.04" y1="71.12" x2="30.48" y2="71.12" width="0.1524" layer="91"/>
+<label x="30.48" y="71.12" size="1.778" layer="95"/>
 </segment>
 </net>
@@
 <segment>
 <pinref part="U$4" gate="G$1" pin="CATHODE"/>
-<wire x1="66.04" y1="66.04" x2="35.56" y2="66.04" width="0.1524" layer="91"/>
-<label x="35.56" y="66.04" size="1.778" layer="95"/>
+<wire x1="66.04" y1="66.04" x2="30.48" y2="66.04" width="0.1524" layer="91"/>
+<label x="30.48" y="66.04" size="1.778" layer="95"/>
+</segment>
+<segment>
+<pinref part="U$3" gate="G$1" pin="GND"/>
+<wire x1="-17.78" y1="25.4" x2="-27.94" y2="25.4" width="0.1524" layer="91"/>
+<label x="-27.94" y="25.4" size="1.778" layer="95"/>
 </segment>
 </net>
@@
 </segment>
 </net>
+<net name="N$10" class="0">
+<segment>
+<pinref part="U$3" gate="G$1" pin="DIR"/>
+<wire x1="-17.78" y1="71.12" x2="-22.86" y2="71.12" width="0.1524" layer="91"/>
+<wire x1="-22.86" y1="71.12" x2="-22.86" y2="73.66" width="0.1524" layer="91"/>
+<wire x1="-22.86" y1="73.66" x2="-27.94" y2="73.66" width="0.1524" layer="91"/>
+</segment>
+</net>
+<net name="+5V" class="0">
+<segment>
+<pinref part="U$3" gate="G$1" pin="VCC"/>
+<wire x1="7.62" y1="71.12" x2="20.32" y2="71.12" width="0.1524" layer="91"/>
+<label x="15.24" y="71.12" size="1.778" layer="95"/>
+</segment>
+</net>
